File: termometer_kombo.kicad_pcb (KiCad board)
At the start: 2 copper layers, 33 x 138 mm, 59 parts, among them J1 USB_B_Micro, J2 Conn_01x04, SW1 SW_MEC, U1 DS18B20, U3 STM32F070F6Px, U4 RT9080, Y1 TBD

Commit message: update
Parts:
- removed the C7 at (112.0, 146.4)
- added FID1: Fiducial_1mm_Mask2mm, Fiducial:Fiducial_1mm_Mask2mm, F.Cu at (115.9, 148.4)
- added FID1: Fiducial_1mm_Mask2mm, Fiducial:Fiducial_1mm_Mask2mm, F.Cu at (115.3, 28.7)
- added FID1: Fiducial_1mm_Mask2mm, Fiducial:Fiducial_1mm_Mask2mm, F.Cu at (87.1, 148.4)
- C5: renamed from C6; value 100µF -> 1µF
- R1, R2, R3, R4, R5, R6: value 120 -> 22
- moved R10 55.6 mm to (113.9, 76.5), turned to 180 degrees
- moved U3 32.5 mm to (110.7, 69.2)
- moved C3 27.8 mm to (109.9, 137.5), turned to 180 degrees
- moved C4 25.4 mm to (109.9, 144.3), turned to 180 degrees
- moved R8 20.7 mm to (114.2, 106.6)
- moved U2 18.6 mm to (109.9, 140.9), turned to 90 degrees
- moved R1 18.2 mm to (109.8, 76.5), turned to 180 degrees
- moved R2 17.7 mm to (109.8, 80.0), turned to 180 degrees
- moved R3 17.1 mm to (109.8, 83.5), turned to 180 degrees
- moved J2 10.2 mm to (116.0, 137.4)
- moved C7 9.49 mm to (109.9, 135.1)
- moved R9 9.23 mm to (107.7, 124.0)
- moved C1 8.95 mm to (111.1, 114.7)
- moved C2 8.95 mm to (111.1, 111.2)
- moved R7 8.95 mm to (111.1, 118.2)
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- renumbered C3 to C1, C5 to C3, C1 to C6, C8 to C7, R8 to R10, R10 to R11, R9 to R7, R7 to R8, R11 to R9, U3 to U1, U4 to U2, U1 to U3
Routing:
- net Net-(D1-A): track 0.00 -> 164.0 mm, vias 0 -> 1
- net Net-(D10-A): track 0.00 -> 129.1 mm
- net Net-(D1-K): track 0.00 -> 127.2 mm
- net Net-(D11-K): track 0.00 -> 112.6 mm
- net Net-(D13-A): track 0.00 -> 95.7 mm
- net IO0: track 0.00 -> 69.4 mm, vias 0 -> 1
- net Net-(D11-A): track 0.00 -> 61.8 mm
- net IO1: track 0.00 -> 56.1 mm, vias 0 -> 2
- net IO2: track 0.00 -> 53.9 mm, vias 0 -> 2
- net IO3: track 0.00 -> 49.3 mm, vias 0 -> 2
- net IO5: track 0.00 -> 47.8 mm, vias 0 -> 2
- net IO4: track 0.00 -> 47.4 mm, vias 0 -> 2
- net IO13: track 0.00 -> 45.2 mm, vias 0 -> 1
- net IO6: track 0.00 -> 44.3 mm, vias 0 -> 2
- net RST: track 0.00 -> 28.0 mm
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- added copper zone on F.Cu, net +3.3V
- added copper zone on F.Cu, net D+
- added copper zone on F.Cu, net D-
- removed copper zone on F.Cu, net GND
Other:
- board text removed: "THT"
