File: termometer_kombo.kicad_sch (KiCad schematic)
At the start: 57 parts, among them J1 USB_B_Micro, J2 Conn_01x04, SW1 SW_MEC, U1 DS18B20, U3 STM32F070F6Px, U4 RT9080, Y1 TBD

Commit message: update
Parts:
- removed C7: 100µF, Capacitor_SMD:C_0805_2012Metric, symbol Device:C_Small
- C5: renamed from C6; value 100µF -> 1µF
- R1, R2, R3, R4, R5, R6: value 120 -> 22
- renumbered C3 to C1, C5 to C3, C1 to C6, C8 to C7, R8 to R10, R10 to R11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
Other:
- moved on the sheet: C6, C7
